File: converter_adapter_ibm4704.kicad_pcb (KiCad board)
At the start: 2 copper layers, 30.5 x 29 mm, 10 parts, among them CN1 MINI_DIN_8P_JACK, P1 CONN_01X10

Commit message: Fix for NEWS
Parts:
- added SJ8: SOLDER_JUMPER, keyboard_parts:SOLDER_JUMPER_2, B.Cu at (96.5, 88.0)
- added SJ9: SOLDER_JUMPER, keyboard_parts:SOLDER_JUMPER_2, B.Cu at (91.5, 88.0)
- G***: footprint keyboard_parts:tmk2016 -> keyboard_parts:tmk_logo
- moved SJ7 9.25 mm to (99.0, 88.0)
- moved SJ5 3.75 mm to (89.0, 88.0)
- moved SJ1 3.25 mm to (103.5, 88.0)
- moved G*** 2.87 mm to (100.7, 76.3)
- moved SJ3 2.75 mm to (106.0, 88.0)
- moved SJ4 2.25 mm to (108.5, 88.0)
- moved SJ2 2.00 mm to (111.0, 88.0)
- moved SJ6 1.75 mm to (94.0, 88.0)
Connections:
- net /D0 renamed /DIN3
- net /D1 renamed /DIN5
- CN1 pad 1: Net-(CN1-Pad1) -> /DIN1
- CN1 pad 6: /VCC -> /DIN6
- CN1 pad 8: GND -> /DIN8
- P1 pad 6: Net-(P1-Pad6) -> /DS_6
- P1 pad 9: /DS_9 -> Net-(P1-Pad9)
- SJ1 pad 1: GND -> /DIN8
- SJ2 pad 1: /VCC -> /DIN6
- SJ5 pad 1: /VCC -> /DIN1
- SJ7 pad 1: GND -> /DIN8
- SJ7 pad 2: /DS_9 -> /DS_5
Routing:
- net /VCC: track 56.1 -> 0.00 mm
- net /DIN6: track 0.00 -> 36.7 mm, vias 0 -> 1
- net /DS_9: track 22.4 -> 0.00 mm
- net /DIN5: track 9.88 -> 29.2 mm, vias 0 -> 1
- net /DIN8: track 0.00 -> 17.9 mm, vias 0 -> 1
- net /DIN1: track 0.00 -> 17.2 mm
- net /DS_5: track 5.17 -> 16.1 mm, vias 0 -> 1
- net /DS_6: track 0.00 -> 10.5 mm
- net /DS_2: track 6.13 -> 13.0 mm
- net /DIN3: track 17.6 -> 23.7 mm
- net /DS_1: track 5.59 -> 8.24 mm
- net GND: track 2.31 -> 0.00 mm, vias 1 -> 0
- net /DS_3: track 26.0 -> 24.2 mm, vias 0 -> 1
- net /DS_4: track 5.08 -> 6.22 mm
